Commit message: feat: robot starts navigating (still nuts)!

File: omniv/launch/fancy_robot.urdf (robot description, URDF)
Before this commit: robot fancy_robot, 5 links, 4 joints
Links:
- removed link left_wheel
- removed link right_wheel
- added link back_left_wheel, mass 0.5; collision cylinder length=0.05 radius=0.1; visual cylinder length=0.05 radius=0.1
- added link back_right_wheel, mass 0.5; collision cylinder length=0.05 radius=0.1; visual cylinder length=0.05 radius=0.1
- added link front_left_wheel, mass 0.5; collision cylinder length=0.05 radius=0.1; visual cylinder length=0.05 radius=0.1
- added link front_right_wheel, mass 0.5; collision cylinder length=0.05 radius=0.1; visual cylinder length=0.05 radius=0.1
Joints:
- removed joint left_wheel_joint
- removed joint right_wheel_joint
- added joint back_left_wheel_joint: type continuous, parent base_link, child back_left_wheel, origin xyz=-0.2 0.225 -0.05 rpy=1.5708 0 0, axis 0 0 1
- added joint back_right_wheel_joint: type continuous, parent base_link, child back_right_wheel, origin xyz=-0.2 -0.225 -0.05 rpy=1.5708 0 0, axis 0 0 1
- added joint front_left_wheel_joint: type continuous, parent base_link, child front_left_wheel, origin xyz=0.2 0.225 -0.05 rpy=1.5708 0 0, axis 0 0 1
- added joint front_right_wheel_joint: type continuous, parent base_link, child front_right_wheel, origin xyz=0.2 -0.225 -0.05 rpy=1.5708 0 0, axis 0 0 1
