Commit message: feat: some enhancement "flies now"!

File: omniv/urdf/limo_ackerman.xacro (robot description, xacro)
@@ -14,5 +14,5 @@
     <xacro:property name="track" value="0.14"/>
     <xacro:property name="wheel_vertical_offset" value="-0.100998" />
-    <xacro:property name="base_mass" value="2.1557"/>
+    <xacro:property name="base_mass" value="1.0"/>
     <xacro:property name="wheel_length" value="0.045" />
     <xacro:property name="wheel_radius" value="0.045" />
@@ -21,5 +21,5 @@
     <parent link="base_footprint"/>
     <child link="base_link"/>
-    <origin xyz="0.0 0.0 0.15" rpy="0 0 0"/>
+    <origin xyz="0.0 0.0 0.055" rpy="0 0 0"/>
     </joint>
     <!-- Base link -->
@@ -83,5 +83,5 @@
         <child link="rear_left_wheel_link"/>
         <origin xyz="${-wheelbase/2} ${track/2} ${wheel_vertical_offset}" rpy="0 0 0" />
-        <axis xyz="0 1 0"/>
+        <axis xyz="0 -1 0"/>
     </joint>
     <link name="rear_right_wheel_link">
@@ -108,5 +108,5 @@
             <child link="rear_right_wheel_link"/>
             <origin xyz="${-wheelbase/2} ${-track/2} ${wheel_vertical_offset}" rpy="${M_PI} 0 0" />
-            <axis xyz="0 -1 0"/>
+            <axis xyz="0 1 0"/>
         </joint>
 </robot>
